File: morserino/morserino.kicad_pcb (KiCad board)
At the start: 2 copper layers, 17 parts, among them J1 encoder, J10 buzzer, J2 paddles, J3 displej, J4 jumper, J5 jumper, J6 LED-R, J7 LED-G, J8 LED-B, J9 buzzer-ext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

Commit message: První návrh PCB.
Parts:
- moved J3 100.1 mm to (36.8, 125.7), turned to 180 degrees
- moved R1 89.8 mm to (48.3, 96.5), turned to 90 degrees
- moved U2 82.1 mm to (52.1, 88.9), turned to 0 degrees
- moved U1 80.4 mm to (42.8, 117.1), turned to 90 degrees
- moved R4 70.0 mm to (67.3, 96.5), turned to 90 degrees
- moved R5 64.9 mm to (72.4, 96.5), turned to 90 degrees
- moved J9 63.6 mm to (62.2, 90.2), turned to 180 degrees
- moved R3 60.0 mm to (77.5, 96.5), turned to 90 degrees
- moved R2 50.4 mm to (87.6, 96.5), turned to 90 degrees
- moved J7 50.2 mm to (67.3, 90.2), turned to 180 degrees
- moved J8 49.7 mm to (72.4, 90.2), turned to 180 degrees
- moved J10 48.8 mm to (82.5, 90.2), turned to 180 degrees
- moved J4 46.1 mm to (62.2, 97.8), turned to 180 degrees
- moved J2 42.8 mm to (97.8, 113.0)
- moved J6 36.9 mm to (77.5, 90.2), turned to 180 degrees
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