File: morserino/morserino.kicad_sch (KiCad schematic)
At the start: 17 parts, among them J1 encoder, J10 buzzer, J2 paddles, J3 displej, J4 jumper, J5 jumper, J6 LED-R, J7 LED-G, J8 LED-B, J9 buzzer-ext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

Commit message: zdroj.
Parts:
- removed J6: LED-R, HAM:PinSocket_1x02_P2.54mm_Vertical_big_pads, symbol Connector:Conn_01x02_Pin
- removed J7: LED-G, HAM:PinSocket_1x02_P2.54mm_Vertical_big_pads, symbol Connector:Conn_01x02_Pin
- removed J8: LED-B, HAM:PinSocket_1x02_P2.54mm_Vertical_big_pads, symbol Connector:Conn_01x02_Pin
- removed R3, R4, R5: 2k7, Resistor_SMD:R_1206_3216Metric_Pad1.30x1.75mm_HandSolder, symbol Device:R
- added D1: WS2812B, HAM:LED_WS2812B-Mini_PLCC4_3.5x3.5mm_bigger_pads, symbol LED:WS2812B
- renumbered J9 to J6, J10 to J7
Connections:
- net GND: now also D1.3 (VSS)
- net +5V: now reaches U1.18 (VIN)
- net +5V: now also D1.1 (VDD)
- net at U1.31 (GPIO19_VSPI-MISO): now also D1.4 (DIN)
Other:
- moved on the sheet: J1, J2
