File: powersourcer/powersourcer/powersourcer.kicad_sch (KiCad schematic)
At the start: 0 parts

Commit message: poslední práce.
Changed lines of the file:
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@@
 	(paper "A4")
 	(sheet
-		(at 104.14 72.39)
+		(at 16.51 19.05)
 		(size 53.34 44.45)
 		(exclude_from_sim no)
@@
 		)
 		(property "Sheetname" "regulace"
-			(at 104.14 71.6784 0)
+			(at 16.51 18.3384 0)
 			(show_name no)
 			(do_not_autoplace no)
@@
 		)
 		(property "Sheetfile" "regulace.kicad_sch"
-			(at 104.14 117.4246 0)
+			(at 16.51 64.0846 0)
 			(show_name no)
 			(do_not_autoplace no)
