File: UV_osvitovka/uv_rizeni/uv_rizeni.kicad_sch (KiCad schematic)
At the start: 11 parts, among them J1 power, J2 UV_switch, K1 FINDER-40.51, SW1 SW_Push, U1 NE555P

Commit message: Přidány kontakty pro externí start tlačítko.
Parts:
- added J3: ext. switch, symbol Connector:Conn_01x02_Socket
Connections:
- net GND: now also J3.1 (Pin_1)
- net at R1.2, SW1.2, U1.2 (TR): now also J3.2 (Pin_2)
Changed lines of the file:
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@@
 	(paper "A4")
 	(junction
+		(at 101.6 88.9)
+		(diameter 0)
+		(color 0 0 0 0)
+	)
+	(junction
 		(at 156.21 73.66)
 		(diameter 0)
@@
 	(wire
 		(pts
-			(xy 101.6 86.36) (xy 101.6 101.6)
+			(xy 101.6 86.36) (xy 101.6 88.9)
 		)
 		(stroke
@@
 	(wire
 		(pts
+			(xy 95.25 82.55) (xy 95.25 88.9)
+		)
+		(stroke
+			(width 0)
+			(type default)
+		)
+	)
+	(wire
+		(pts
+			(xy 95.25 80.01) (xy 95.25 73.66)
+		)
+		(stroke
+			(width 0)
+			(type default)
+		)
+	)
+	(wire
+		(pts
 			(xy 110.49 78.74) (xy 110.49 90.17)
 		)
@@
 	(wire
 		(pts
+			(xy 95.25 73.66) (xy 101.6 73.66)
+		)
+		(stroke
+			(width 0)
+			(type default)
+		)
+	)
+	(wire
+		(pts
 			(xy 181.61 58.42) (xy 181.61 80.01)
 		)
@@
 	(wire
 		(pts
+			(xy 90.17 82.55) (xy 95.25 82.55)
+		)
+		(stroke
+			(width 0)
+			(type default)
+		)
+	)
+	(wire
+		(pts
 			(xy 110.49 101.6) (xy 101.6 101.6)
 		)
@@
 	(wire
 		(pts
+			(xy 95.25 88.9) (xy 101.6 88.9)
+		)
+		(stroke
+			(width 0)
+			(type default)
+		)
+	)
+	(wire
+		(pts
 			(xy 191.77 97.79) (xy 184.15 97.79)
 		)
@@
 	(wire
 		(pts
+			(xy 90.17 80.01) (xy 95.25 80.01)
+		)
+		(stroke
+			(width 0)
+			(type default)
+		)
+	)
+	(wire
+		(pts
 			(xy 156.21 73.66) (xy 156.21 83.82)
 		)
@@
 	(wire
 		(pts
+			(xy 101.6 88.9) (xy 101.6 101.6)
+		)
+		(stroke
+			(width 0)
+			(type default)
+		)
+	)
+	(wire
+		(pts
 			(xy 45.72 29.21) (xy 45.72 31.75)
 		)
@@
 		)
 	)
+	(symbol
+		(lib_id "Connector:Conn_01x02_Socket")
+		(at 85.09 82.55 180)
+		(unit 1)
+		(body_style 1)
+		(exclude_from_sim no)
+		(in_bom yes)
+		(on_board yes)
+		(in_pos_files yes)
+		(dnp no)
+		(fields_autoplaced yes)
+		(property "Reference" "J3"
+			(at 85.725 74.93 0)
+			(show_name no)
+			(do_not_autoplace no)
+			(effects
+				(font
+					(size 1.27 1.27)
+				)
+			)
+		)
+		(property "Value" "ext. switch"
+			(at 85.725 77.47 0)
+			(show_name no)
+			(do_not_autoplace no)
+			(effects
+				(font
+					(size 1.27 1.27)
+				)
+			)
+		)
+		(property "Footprint" ""
+			(at 85.09 82.55 0)
+			(hide yes)
+			(show_name no)
+			(do_not_autoplace no)
+			(effects
+				(font
+					(size 1.27 1.27)
+				)
+			)
+		)
+		(property "Datasheet" ""
+			(at 85.09 82.55 0)
+			(hide yes)
+			(show_name no)
+			(do_not_autoplace no)
+			(effects
+				(font
+					(size 1.27 1.27)
+				)
+			)
+		)
+		(property "Description" "Generic connector, single row, 01x02, script generated"
+			(at 85.09 82.55 0)
+			(hide yes)
+			(show_name no)
+			(do_not_autoplace no)
+			(effects
+				(font
+					(size 1.27 1.27)
+				)
+			)
+		)
+		(pin "1"
+		)
+		(pin "2"
+		)
+		(instances
+			(project "uv_rizeni"
+				(path "/88ef6dbc-0d58-4fd4-a096-6feaeb149775"
+					(reference "J3")
+					(unit 1)
+				)
+			)
+		)
+	)
