File: UV_osvitovka/uv_rizeni/uv_rizeni.kicad_pcb (KiCad board)
At the start: 2 copper layers, 14 parts, among them J1 power, J2 ext. switch, J3 UV_switch, K1 FINDER-40.51, SW1 SW_Push, U1 NE555P

Commit message: rozdýchávání knihovny, ale šlo to.
Parts:
- removed the K1 at (105.0, 59.8)
- removed the R3 at (92.1, 45.7)
- added C1: 100n, HAM_Lib:C_Disc_D10.5mm_W5.0mm_P5.00mm, F.Cu at (181.0, 64.7)
- added C2: 1000uF, HAM_Lib:CP_Radial_D10.0mm_P5.00mm, F.Cu at (187.0, 74.5)
- added D1: LED, HAM:PinHeader_1x02_P2.54mm_Vertical, F.Cu at (170.8, 63.5)
- added D1: LED, HAM:PinHeader_1x02_P2.54mm_Vertical, F.Cu at (83.8, 41.3)
- added J1: power, HAM_Lib:TerminalBlock_CUI_TB007-508-02_1x02_P5.08mm_Horizontal, F.Cu at (169.5, 79.4)
- added J2: ext. switch, HAM_Lib:PinSocket_1x02_P2.54mm_Vertical_big_pads, F.Cu at (210.2, 76.9)
- added J3: UV_switch, HAM_Lib:TerminalBlock_CUI_TB007-508-03_1x03_P5.08mm_Horizontal, F.Cu at (169.5, 49.5)
- added K1: FINDER-40.51, HAM_Lib:Relay_Tyco_Schrack, F.Cu at (99.0, 74.9)
- added K1: FINDER-40.51, HAM_Lib:Relay_Tyco_Schrack, F.Cu at (204.4, 48.3)
- added R1: 10k, Resistor_SMD:R_1206_3216Metric_Pad1.30x1.75mm_HandSolder, B.Cu at (199.4, 66.0)
- added R2: 22k, Resistor_SMD:R_1206_3216Metric_Pad1.30x1.75mm_HandSolder, B.Cu at (191.5, 74.9)
- added R3: 2k7, Resistor_SMD:R_1206_3216Metric_Pad1.30x1.75mm_HandSolder, B.Cu at (90.2, 41.3)
- added R3: 2k7, Resistor_SMD:R_1206_3216Metric_Pad1.30x1.75mm_HandSolder, B.Cu at (170.8, 57.1)
- added RV1: 100k, HAM_Lib:Potentiometer_Bourns_3296W_Vertical, F.Cu at (197.8, 74.3)
- added SW1: SW_Push, HAM_Lib:SW_PUSH_6mm_H5mm, F.Cu at (211.2, 59.0)
- added U1: NE555P, HAM_Lib:DIP-8_W7.62mm, F.Cu at (194.9, 58.4)
- D2: value LED -> 1N4007; footprint HAM_Lib:PinSocket_1x02_P2.54mm_Vertical_big_pads -> HAM_Lib:D_DO-41_SOD81_P10.16mm_Horizontal
- moved D2 125.8 mm to (210.8, 49.5)
- moved J2 36.5 mm to (70.5, 80.6), turned to 180 degrees
- moved D2 22.9 mm to (97.8, 81.3), turned to 0 degrees
- moved J3 19.9 mm to (97.8, 40.0)
- moved R2 8.64 mm to (72.4, 61.9)
- moved RV1 8.52 mm to (73.0, 68.3)
- moved R1 7.41 mm to (81.3, 69.8)
- moved J1 6.25 mm to (67.9, 40.0)
- moved C1 6.02 mm to (82.6, 51.4)
- moved C2 5.70 mm to (72.9, 57.5)
- moved U1 4.84 mm to (88.9, 65.4)
- moved SW1 2.69 mm to (88.3, 81.6)
- renumbered D1 to D2
Connections:
- D2 pad 1: Net-(D1-K) -> Net-(D2-K)
- D2 pad 1: GND -> Net-(D2-K)
- D2 pad 2: Net-(D2-A) -> GND
- U1 pad 3: Net-(D1-K) -> Net-(D2-K)
Routing:
- net GND: track 140.7 -> 275.5 mm
- net +12V: track 146.1 -> 245.7 mm
- net Net-(D2-K): track 0.00 -> 95.7 mm
- net Net-(J2-Pin_2): track 31.4 -> 78.3 mm
- net Net-(D1-K): track 33.1 -> 0.00 mm
- net Net-(J3-Pin_1): track 22.8 -> 43.6 mm
- net Net-(U1-DIS): track 17.9 -> 29.1 mm
- net Net-(R2-Pad1): track 6.70 -> 17.0 mm
- net Net-(J3-Pin_3): track 22.8 -> 31.4 mm
- net Net-(U1-CV): track 5.62 -> 13.8 mm
- net Net-(D1-A): track 0.00 -> 4.53 mm
- net Net-(D2-A): track 2.90 -> 0.00 mm
- removed copper zone on B.Cu, net GND
