File: UV_osvitovka/uv_rizeni/uv_rizeni-backups/uv_rizeni-2026-04-30_134258/uv_rizeni.kicad_sch (KiCad schematic)
At the start: 14 parts, among them J1 power, J2 ext. switch, J3 UV_switch, K1 FINDER-40.51, SW1 SW_Push, U1 NE555P

Commit message: Celý se to posralo kvůli chybějícímu řádku.
Parts:
- D2: renamed from D1; footprint HAM:PinHeader_1x02_P2.54mm_Vertical -> (none)
- R2: footprint Resistor_SMD:R_1206_3216Metric_Pad1.30x1.75mm_HandSolder -> HAM_Lib:R_Axial_DIN0309_L9.0mm_D3.2mm_P12.70mm_Horizontal
- R3: footprint Resistor_SMD:R_1206_3216Metric_Pad1.30x1.75mm_HandSolder -> (none)
- renumbered D2 to D1
Changed lines of the file:
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@@
 			)
 		)
-		(property "Footprint" "Resistor_SMD:R_1206_3216Metric_Pad1.30x1.75mm_HandSolder"
+		(property "Footprint" ""
 			(at 159.512 81.28 90)
 			(hide yes)
@@
 		(dnp no)
 		(fields_autoplaced yes)
-		(property "Reference" "D1"
+		(property "Reference" "D2"
 			(at 165.1 93.0274 90)
 			(show_name no)
@@
 			)
 		)
-		(property "Footprint" "HAM:PinHeader_1x02_P2.54mm_Vertical"
+		(property "Footprint" ""
 			(at 161.29 92.71 0)
 			(hide yes)
@@
 			(project "uv_rizeni"
 				(path "/88ef6dbc-0d58-4fd4-a096-6feaeb149775"
-					(reference "D1")
+					(reference "D2")
 					(unit 1)
 				)
@@
 			)
 		)
-		(property "Footprint" "Resistor_SMD:R_1206_3216Metric_Pad1.30x1.75mm_HandSolder"
+		(property "Footprint" "HAM_Lib:R_Axial_DIN0309_L9.0mm_D3.2mm_P12.70mm_Horizontal"
 			(at 141.732 67.31 90)
 			(hide yes)
@@
 		(dnp no)
 		(fields_autoplaced yes)
-		(property "Reference" "D2"
+		(property "Reference" "D1"
 			(at 176.53 86.3599 90)
 			(show_name no)
@@
 			(project "uv_rizeni"
 				(path "/88ef6dbc-0d58-4fd4-a096-6feaeb149775"
-					(reference "D2")
-					(unit 1)
-				)
+					(reference "D1")
+					(unit 1)
+				)
